Commit message: fixed slam toolbox for single robot with namespace

File: src/autobot/description/gazebo_control.xacro (robot description, xacro)
@@ -17,5 +17,5 @@
                 <max_wheel_acceleration>10.0</max_wheel_acceleration>
                 <odometry_frame>${robot_name}/odom</odometry_frame>
-                <robot_base_frame>${robot_name}/base_link</robot_base_frame>
+                <robot_base_frame>${robot_name}/base_footprint</robot_base_frame>
                 <publish_odom>true</publish_odom>
                 <publish_odom_tf>true</publish_odom_tf>

File: src/autobot/description/lidar.xacro (robot description, xacro)
@@ -3,5 +3,5 @@
     <xacro:macro name="lidar" params="robot_name">
         <joint name="laser_joint" type="fixed">
-            <parent link="chassis"/>
+            <parent link="base_link"/>
             <child link="laser_frame"/>
             <origin xyz="0.122 0 0.212" rpy="0 0 0"/>

File: src/autobot/description/robot_core.xacro (robot description, xacro)
@@ -13,5 +13,5 @@
         <xacro:property name="wheel_offset_x" value="0.226"/>
         <xacro:property name="wheel_offset_y" value="0.1485"/>
-        <xacro:property name="wheel_offset_z" value="0.01"/>
+        <xacro:property name="wheel_offset_z" value="0.00"/>
         <xacro:property name="caster_wheel_radius" value="0.015"/>
         <xacro:property name="caster_wheel_mass" value="0.01"/>
@@ -33,22 +33,20 @@
             <color rgba="1 0 0 1"/>
         </material>
+        <!-- BASE_FOOTPRINT LINK -->
+        <link name="base_footprint"/>
+        <joint name="base_joint" type="fixed">
+            <parent link="base_footprint"/>
+            <child link="base_link"/>
+            <origin xyz="0.0 0.0 0.010" rpy="0 0 0"/>
+        </joint>
         <!-- BASE LINK -->
-        <link name="base_link">
+        <!-- <link name="base_link">
         </link>
-        <!-- BASE_FOOTPRINT LINK -->
-        <joint name="base_footprint_joint" type="fixed">
-            <parent link="base_link"/>
-            <child link="base_footprint"/>
-            <origin xyz="0 0 0" rpy="0 0 0"/>
-        </joint>
-        <link name="base_footprint">
-        </link>
-        <!-- CHASSIS LINK -->
         <joint name="chassis_joint" type="fixed">
             <parent link="base_link"/>
             <child link="chassis"/>
             <origin xyz="${-wheel_offset_x} 0 ${-wheel_offset_z}"/>
-        </joint>
-        <link name="chassis">
+        </joint> -->
+        <link name="base_link">
             <visual>
                 <origin xyz="${chassis_length/2} 0 ${chassis_height/2}"/>
@@ -68,5 +66,5 @@
             </xacro:inertial_box>
         </link>
-        <gazebo reference="chassis">
+        <gazebo reference="base_link">
             <material>Gazebo/Blue</material>
         </gazebo>
@@ -75,5 +73,5 @@
             <parent link="base_link"/>
             <child link="left_wheel"/>
-            <origin xyz="0 ${wheel_offset_y} 0" rpy="-${pi/2} 0 0" />
+            <origin xyz="0.22 ${wheel_offset_y} 0" rpy="-${pi/2} 0 0" />
             <axis xyz="0 0 1"/>
         </joint>
@@ -101,5 +99,5 @@
             <parent link="base_link"/>
             <child link="right_wheel"/>
-            <origin xyz="0 ${-wheel_offset_y} 0" rpy="${pi/2} 0 0" />
+            <origin xyz="0.22 ${-wheel_offset_y} 0" rpy="${pi/2} 0 0" />
             <axis xyz="0 0 -1"/>
         </joint>
@@ -125,5 +123,5 @@
         <!-- CASTER WHEEL LINK -->
         <joint name="caster_wheel_joint" type="fixed">
-            <parent link="chassis"/>
+            <parent link="base_link"/>
             <child link="caster_wheel"/>
             <origin xyz="${caster_wheel_offset_x} 0 ${caster_wheel_offset_z}"/>
